Commit message: Clean up redis client a bit, and factor out EE link name

File: src/controller/kuka_iiwa.urdf (robot description, URDF)
Before this commit: robot kuka_iiwa, 8 links, 7 joints
Links:
- removed link link6
- added link EE, mass 1; collision mesh filename=kuka_iiwa_graphics/link6.obj scale=1 1 1; visual mesh filename=kuka_iiwa_graphics/link6.obj scale=1 1 1
Joints:
- joint j6: child link6 -> EE
